Commit message: gitignore added

File: catkin_larc/src/navigation/robot_description/urdf/nexus_4wd_mecanum.xacro (robot description, xacro)
@@ -6,6 +6,8 @@
   <material name="yellow"><color rgba="0.8 0.8 0.0 1.0" /></material>
   <material name="black"><color rgba="0.15 0.15 0.15 1.0" /></material>
+  <material name="Black"><color rgba="0.15 0.15 0.15 1.0" /></material>
   <material name="dark_grey"><color rgba="0.2 0.2 0.2 1.0" /></material>
   <material name="light_grey"><color rgba="0.4 0.4 0.4 1.0" /></material>
+  <virtual_joint name="world_joint" type="planar" parent_frame="odom" child_link="base_footprint"/>
   <link name="base_footprint"></link>
   <joint name="base_link_joint" type="fixed">
@@ -18,5 +20,5 @@
       <origin xyz="0 0 0" rpy="0 0 0" />
       <geometry>
-        <mesh filename="package://nexus_4wd_mecanum_description/meshes/nexus_base_link.STL" scale="0.001 0.001 0.001"/>
+        <mesh filename="package://robot_description/meshes/nexus/nexus_base_link.STL" scale="0.001 0.001 0.001"/>
       </geometry>
       <material name="yellow" />
@@ -25,5 +27,5 @@
       <origin xyz="0 0 0"/>
       <geometry>
-        <mesh filename="package://nexus_4wd_mecanum_description/meshes/nexus_base_link_collision.STL" scale="0.001 0.001 0.001"/>
+        <mesh filename="package://robot_description/meshes/nexus/nexus_base_link_collision.STL" scale="0.001 0.001 0.001"/>
       </geometry>
     </collision>
@@ -47,12 +49,12 @@
       <origin xyz="0 0 0" rpy="0 0 0" />
       <geometry>
-        <mesh filename="package://nexus_4wd_mecanum_description/meshes/wheel_shaft.STL" scale="0.001 0.001 0.001"/>
-      </geometry>
-      <material name="black" />
-    </visual>
-    <collision>
-      <origin xyz="0 0 0"/>
-      <geometry>
-        <mesh filename="package://nexus_4wd_mecanum_description/meshes/wheel_shaft.STL" scale="0.001 0.001 0.001"/>
+        <mesh filename="package://robot_description/meshes/nexus/wheel_shaft.STL" scale="0.001 0.001 0.001"/>
+      </geometry>
+      <material name="black" />
+    </visual>
+    <collision>
+      <origin xyz="0 0 0"/>
+      <geometry>
+        <mesh filename="package://robot_description/meshes/nexus/wheel_shaft.STL" scale="0.001 0.001 0.001"/>
       </geometry>
     </collision>
@@ -75,12 +77,12 @@
       <origin xyz="0 0 0" rpy="0 0 0" />
       <geometry>
-        <mesh filename="package://nexus_4wd_mecanum_description/meshes/wheel_shaft.STL" scale="0.001 0.001 0.001"/>
-      </geometry>
-      <material name="black" />
-    </visual>
-    <collision>
-      <origin xyz="0 0 0"/>
-      <geometry>
-        <mesh filename="package://nexus_4wd_mecanum_description/meshes/wheel_shaft.STL" scale="0.001 0.001 0.001"/>
+        <mesh filename="package://robot_description/meshes/nexus/wheel_shaft.STL" scale="0.001 0.001 0.001"/>
+      </geometry>
+      <material name="black" />
+    </visual>
+    <collision>
+      <origin xyz="0 0 0"/>
+      <geometry>
+        <mesh filename="package://robot_description/meshes/nexus/wheel_shaft.STL" scale="0.001 0.001 0.001"/>
       </geometry>
     </collision>
@@ -103,12 +105,12 @@
       <origin xyz="0 0 0" rpy="0 0 0" />
       <geometry>
-        <mesh filename="package://nexus_4wd_mecanum_description/meshes/wheel_shaft.STL" scale="0.001 0.001 0.001"/>
-      </geometry>
-      <material name="black" />
-    </visual>
-    <collision>
-      <origin xyz="0 0 0"/>
-      <geometry>
-        <mesh filename="package://nexus_4wd_mecanum_description/meshes/wheel_shaft.STL" scale="0.001 0.001 0.001"/>
+        <mesh filename="package://robot_description/meshes/nexus/wheel_shaft.STL" scale="0.001 0.001 0.001"/>
+      </geometry>
+      <material name="black" />
+    </visual>
+    <collision>
+      <origin xyz="0 0 0"/>
+      <geometry>
+        <mesh filename="package://robot_description/meshes/nexus/wheel_shaft.STL" scale="0.001 0.001 0.001"/>
       </geometry>
     </collision>
@@ -131,12 +133,12 @@
       <origin xyz="0 0 0" rpy="0 0 0" />
       <geometry>
-        <mesh filename="package://nexus_4wd_mecanum_description/meshes/wheel_shaft.STL" scale="0.001 0.001 0.001"/>
-      </geometry>
-      <material name="black" />
-    </visual>
-    <collision>
-      <origin xyz="0 0 0"/>
-      <geometry>
-        <mesh filename="package://nexus_4wd_mecanum_description/meshes/wheel_shaft.STL" scale="0.001 0.001 0.001"/>
+        <mesh filename="package://robot_description/meshes/nexus/wheel_shaft.STL" scale="0.001 0.001 0.001"/>
+      </geometry>
+      <material name="black" />
+    </visual>
+    <collision>
+      <origin xyz="0 0 0"/>
+      <geometry>
+        <mesh filename="package://robot_description/meshes/nexus/wheel_shaft.STL" scale="0.001 0.001 0.001"/>
       </geometry>
     </collision>
@@ -160,5 +162,5 @@
       <origin xyz="0 0 0" rpy="0 0 0" />
       <geometry>
-        <mesh filename="package://nexus_4wd_mecanum_description/meshes/mecanum_wheel_left.STL" scale="0.001 0.001 0.001"/>
+        <mesh filename="package://robot_description/meshes/nexus/mecanum_wheel_left.STL" scale="0.001 0.001 0.001"/>
       </geometry>
       <material name="light_grey" />
@@ -190,5 +192,5 @@
       <origin xyz="0 0 0" rpy="0 0 0" />
       <geometry>
-        <mesh filename="package://nexus_4wd_mecanum_description/meshes/mecanum_wheel_right.STL" scale="0.001 0.001 0.001"/>
+        <mesh filename="package://robot_description/meshes/nexus/mecanum_wheel_right.STL" scale="0.001 0.001 0.001"/>
       </geometry>
       <material name="light_grey" />
@@ -220,5 +222,5 @@
       <origin xyz="0 0 0" rpy="0 0 0" />
       <geometry>
-        <mesh filename="package://nexus_4wd_mecanum_description/meshes/mecanum_wheel_right.STL" scale="0.001 0.001 0.001"/>
+        <mesh filename="package://robot_description/meshes/nexus/mecanum_wheel_right.STL" scale="0.001 0.001 0.001"/>
       </geometry>
       <material name="light_grey" />
@@ -250,5 +252,5 @@
       <origin xyz="0 0 0" rpy="0 0 0" />
       <geometry>
-        <mesh filename="package://nexus_4wd_mecanum_description/meshes/mecanum_wheel_left.STL" scale="0.001 0.001 0.001"/>
+        <mesh filename="package://robot_description/meshes/nexus/mecanum_wheel_left.STL" scale="0.001 0.001 0.001"/>
       </geometry>
       <material name="light_grey" />
@@ -279,5 +281,5 @@
       <origin xyz="0 0 0" rpy="${PI/2} 0 0" />
       <geometry>
-        <mesh filename="package://nexus_4wd_mecanum_description/meshes/urm04.STL" scale="0.001 0.001 0.001"/>
+        <mesh filename="package://robot_description/meshes/nexus/urm04.STL" scale="0.001 0.001 0.001"/>
       </geometry>
       <material name="black" />
@@ -293,5 +295,5 @@
       <origin xyz="0 0 0" rpy="${PI/2} 0 0" />
       <geometry>
-        <mesh filename="package://nexus_4wd_mecanum_description/meshes/urm04.STL" scale="0.001 0.001 0.001"/>
+        <mesh filename="package://robot_description/meshes/nexus/urm04.STL" scale="0.001 0.001 0.001"/>
       </geometry>
       <material name="black" />
@@ -307,5 +309,5 @@
       <origin xyz="0 0 0" rpy="${PI/2} 0 0" />
       <geometry>
-        <mesh filename="package://nexus_4wd_mecanum_description/meshes/urm04.STL" scale="0.001 0.001 0.001"/>
+        <mesh filename="package://robot_description/meshes/nexus/urm04.STL" scale="0.001 0.001 0.001"/>
       </geometry>
       <material name="black" />
@@ -321,44 +323,38 @@
       <origin xyz="0 0 0" rpy="${PI/2} 0 0" />
       <geometry>
-        <mesh filename="package://nexus_4wd_mecanum_description/meshes/urm04.STL" scale="0.001 0.001 0.001"/>
-      </geometry>
-      <material name="black" />
-    </visual>
-  </link>
-  <gazebo reference="base_scan">
-    <sensor type="ray" name="head_rplidar_sensor">
-      <pose>0 0 0.06 0 0 0</pose>
-      <visualize>false</visualize>
-      <update_rate>40</update_rate>
-      <ray>
-        <scan>
-          <horizontal>
-            <samples>720</samples>
-            <resolution>1</resolution>
-            <min_angle>-3.14159265</min_angle>
-            <max_angle>3.14159265</max_angle>
-          </horizontal>
-        </scan>
-        <range>
-          <min>0.2</min>
-          <max>12.0</max>
-          <resolution>0.01</resolution>
-        </range>
-        <noise>
-          <type>gaussian</type>
-          <mean>0.0</mean>
-          <stddev>0.01</stddev>
-        </noise>
-      </ray>
-      <plugin name="gazebo_ros_head_rplidar_controller" filename="libgazebo_ros_laser.so">
-        <topicName>scan</topicName>
-        <frameName>base_scan</frameName>
-      </plugin>
-    </sensor>
-  </gazebo>
+        <mesh filename="package://robot_description/meshes/nexus/urm04.STL" scale="0.001 0.001 0.001"/>
+      </geometry>
+      <material name="black" />
+    </visual>
+  </link>
+  <joint name="rplidar_joint" type="fixed">
+    <origin xyz="0.02 0 0.07" rpy="0 0 0"/>
+    <parent link="base_link"/>
+    <child link="base_scan"/>
+  </joint>
+  <!-- rplidar Laser -->
+  <link name="base_scan">
+    <collision>
+      <geometry>
+        <mesh filename="package://robot_description/meshes/rosbot/rplidar.stl" scale="0.001 0.001 0.001" />
+      </geometry>
+    </collision>
+    <visual>
+      <origin xyz="0 0 0" rpy="1.5707 0 4.71"/>
+      <geometry>
+        <mesh filename="package://robot_description/meshes/rosbot/rplidar.stl" scale="0.001 0.001 0.001" />
+      </geometry>
+      <material name="black"/>
+    </visual>
+    <inertial>
+      <mass value="1e-5" />
+      <origin xyz="0 0 0" rpy="0 0 0"/>
+      <inertia ixx="0" ixy="0" ixz="0" iyy="0" iyz="0" izz="0" />
+    </inertial>
+  </link>
   <!-- Include controller plugin for Gazebo -->
-  <xacro:include filename="$(find nexus_4wd_mecanum_description)/urdf/nexus_4wd_mecanum.gazebo" />
+  <xacro:include filename="$(find robot_description)/urdf/nexus_4wd_mecanum.gazebo.xacro" />
   <!-- Include URM04 ultrasonic range finders -->
-  <xacro:include filename="$(find nexus_4wd_mecanum_description)/urdf/urm04_sensor.xacro"/>
+  <xacro:include filename="$(find robot_description)/urdf/urm04_sensor.gazebo.xacro"/>
   <!-- front sensor -->
   <xacro:urm04_sensor frame_name="front_sensor" ros_topic="front_sensor" update_rate="10" min_range="0.04" max_range="2.5" horizontal_field_of_view="1.04" vertical_field_of_view="0.04" ray_count="2" />

Commit message: Lidar localization tests sim

File: catkin_larc/src/navigation/robot_description/urdf/nexus_4wd_mecanum.xacro (robot description, xacro)
@@ -329,5 +329,5 @@
   </link>
   <joint name="rplidar_joint" type="fixed">
-    <origin xyz="0.02 0 0.07" rpy="0 0 0"/>
+    <origin xyz="0.02 0 0.057" rpy="0 0 0"/>
     <parent link="base_link"/>
     <child link="base_scan"/>
